File: Hardware/touch_RevA/TouchBoardSchematic.sch (EAGLE design)
At the start: 14 parts, among them IC1 AT42QT1070-SSU

Commit message: TouchBoard
Routed; version 1
Parts:
- added CHANGE_PIN: (no value), pinhead:PINHD-1X1
- R1, R2, R3, R4, R5: value (none) -> 20k
Connections:
- removed net N$1: IC1.OUT4, R5.1
- new net CHANGE: CHANGE_PIN.1, IC1.OUT4, R5.1
Other:
- moved on the sheet: R5
Changed lines of the file:
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@@
 <part name="C1" library="eagle-ltspice" deviceset="C" device="C0603" value="0.1u"/>
 <part name="GND3" library="supply1" deviceset="GND" device=""/>
-<part name="R1" library="eagle-ltspice" deviceset="R" device="R0603"/>
-<part name="R2" library="eagle-ltspice" deviceset="R" device="R0603"/>
-<part name="R3" library="eagle-ltspice" deviceset="R" device="R0603"/>
-<part name="R4" library="eagle-ltspice" deviceset="R" device="R0603"/>
+<part name="R1" library="eagle-ltspice" deviceset="R" device="R0603" value="20k"/>
+<part name="R2" library="eagle-ltspice" deviceset="R" device="R0603" value="20k"/>
+<part name="R3" library="eagle-ltspice" deviceset="R" device="R0603" value="20k"/>
+<part name="R4" library="eagle-ltspice" deviceset="R" device="R0603" value="20k"/>
 <part name="PWR" library="pinhead" deviceset="PINHD-1X4" device=""/>
 <part name="MICRO" library="pinhead" deviceset="PINHD-1X6" device=""/>
@@
 <part name="TO_TOUCH" library="pinhead" deviceset="PINHD-1X1" device=""/>
 <part name="P+1" library="supply1" deviceset="VCC" device=""/>
+<part name="CHANGE_PIN" library="pinhead" deviceset="PINHD-1X1" device=""/>
+<part name="R5" library="eagle-ltspice" deviceset="R" device="R0603" value="20k"/>
 <part name="P+2" library="supply1" deviceset="VCC" device=""/>
-<part name="R5" library="eagle-ltspice" deviceset="R" device="R0603"/>
 </parts>
 <sheets>
@@
 <instance part="TO_TOUCH" gate="G$1" x="25.4" y="88.9" rot="R90"/>
 <instance part="P+1" gate="VCC" x="48.26" y="53.34"/>
-<instance part="P+2" gate="VCC" x="109.22" y="58.42"/>
-<instance part="R5" gate="G$1" x="99.06" y="53.34"/>
+<instance part="CHANGE_PIN" gate="G$1" x="43.18" y="88.9" rot="R90"/>
+<instance part="R5" gate="G$1" x="116.84" y="48.26" rot="R90"/>
+<instance part="P+2" gate="VCC" x="116.84" y="55.88"/>
 </instances>
 <busses>
@@
 </segment>
 <segment>
-<pinref part="P+2" gate="VCC" pin="VCC"/>
-<pinref part="R5" gate="G$1" pin="2"/>
-<wire x1="104.14" y1="53.34" x2="109.22" y2="53.34" width="0.1524" layer="91"/>
-<wire x1="109.22" y1="53.34" x2="109.22" y2="55.88" width="0.1524" layer="91"/>
-</segment>
-<segment>
 <pinref part="IC1" gate="G$1" pin="!RST"/>
 <pinref part="P+1" gate="VCC" pin="VCC"/>
@@
 <wire x1="48.26" y1="48.26" x2="48.26" y2="50.8" width="0.1524" layer="91"/>
 </segment>
-</net>
-<net name="N$1" class="0">
-<segment>
+<segment>
+<wire x1="50.8" y1="53.34" x2="48.26" y2="53.34" width="0.1524" layer="91"/>
+</segment>
+<segment>
+<pinref part="R5" gate="G$1" pin="2"/>
+<pinref part="P+2" gate="VCC" pin="VCC"/>
+<wire x1="116.84" y1="53.34" x2="116.84" y2="50.8" width="0.1524" layer="91"/>
+</segment>
+</net>
+<net name="CHANGE" class="0">
+<segment>
+<pinref part="CHANGE_PIN" gate="G$1" pin="1"/>
+<wire x1="43.18" y1="86.36" x2="43.18" y2="76.2" width="0.1524" layer="91"/>
+<label x="43.18" y="76.2" size="1.778" layer="95"/>
+</segment>
+<segment>
+<wire x1="101.6" y1="40.64" x2="116.84" y2="40.64" width="0.1524" layer="91"/>
+<pinref part="R5" gate="G$1" pin="1"/>
+<wire x1="116.84" y1="40.64" x2="116.84" y2="43.18" width="0.1524" layer="91"/>
 <pinref part="IC1" gate="G$1" pin="OUT4"/>
-<pinref part="R5" gate="G$1" pin="1"/>
-<wire x1="93.98" y1="53.34" x2="88.9" y2="53.34" width="0.1524" layer="91"/>
-</segment>
-</net>
+<wire x1="88.9" y1="53.34" x2="101.6" y2="53.34" width="0.1524" layer="91"/>
+<wire x1="101.6" y1="53.34" x2="101.6" y2="40.64" width="0.1524" layer="91"/>
+<label x="99.06" y="53.34" size="1.778" layer="95"/>
+</segment>
+</net>
