File: Hardware/touch_RevA/TouchBoardSchematic.brd (EAGLE design)
At the start: 100 x 80 mm, 15 parts, among them IC1 AT42QT1070-SSU

Commit message: Added a bunch of gerbers, and some minor changes
And a bunch of pictures of gerbers
Parts:
- moved LED1 27.2 mm to (25.0, 39.9)
- moved LED2 27.2 mm to (11.0, 14.5)
- moved MICRO 27.2 mm to (31.6, 19.3)
- moved C1 27.2 mm to (22.6, 14.2)
- moved CHANGE_PIN 27.2 mm to (39.1, 33.3)
- moved LED3 27.2 mm to (39.0, 14.5)
- moved R2 27.2 mm to (14.1, 30.4)
- moved R3 27.2 mm to (17.1, 33.2)
- moved R5 27.2 mm to (33.0, 29.1)
- moved ACCEL 27.2 mm to (26.1, 30.5)
- moved IC1 27.2 mm to (23.8, 24.1)
- moved PWR 27.2 mm to (16.9, 20.2)
- moved R1 27.2 mm to (11.1, 27.8)
- moved R4 27.2 mm to (19.8, 35.7)
- moved TO_TOUCH 27.2 mm to (16.9, 38.5)
Other:
- board size 100 x 80 mm -> 50 x 50 mm
