File: Hardware/touch_RevA/touch_RevA.brd (EAGLE design)
At the start: 50 x 50 mm, 15 parts, among them IC1 AT42QT1070-SSU

Commit message: Update of hw files
Added logo to brds, added +/- to LEDs and generated and updated gerber
files.
Other:
- outline, holes or cut-outs redrawn
- board text added: "+"
- board text added: "-"
