File: Hardware/micro_RevA/micro_RevA.sch (EAGLE design)
At the start: 22 parts, among them IC1 TLC59711, Q1 CSTCR6M00G53Z

Commit message: WOW!! Almost forgot to connect data and clk lines
Good to catch the stupid shit early on.
Connections:
- net CLK: now also U$1.PB7(OC0A/OC1C/RTS)
- net DATA: now also U$1.PB6(OC1B/OC4B/ADC13)
Changed lines of the file:
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@@
 <label x="50.8" y="35.56" size="1.778" layer="95"/>
+</segment>
+<segment>
+<pinref part="U$1" gate="G$1" pin="PB7(OC0A/OC1C/RTS)"/>
+<wire x1="129.54" y1="104.14" x2="142.24" y2="104.14" width="0.1524" layer="91"/>
+<label x="137.16" y="104.14" size="1.778" layer="95"/>
 </segment>
 </net>
@@
 <label x="50.8" y="33.02" size="1.778" layer="95"/>
 </segment>
+<segment>
+<pinref part="U$1" gate="G$1" pin="PB6(OC1B/OC4B/ADC13)"/>
+<wire x1="129.54" y1="101.6" x2="142.24" y2="101.6" width="0.1524" layer="91"/>
+<label x="137.16" y="101.6" size="1.778" layer="95"/>
+</segment>
 </net>

Commit message: Completed routing of microcontroller board
Everything is routed and passes drc. Still needs visual inspection.
Connections:
- net VCC: now also U$1./RESET, U$1.AVCC, U$1.AVCC1, U$1.UVCC, U$1.VCC
Changed lines of the file:
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@@
 <segment>
 <pinref part="P+4" gate="VCC" pin="VCC"/>
-<wire x1="83.82" y1="124.46" x2="76.2" y2="124.46" width="0.1524" layer="91"/>
+<wire x1="83.82" y1="124.46" x2="81.28" y2="124.46" width="0.1524" layer="91"/>
+<wire x1="81.28" y1="124.46" x2="76.2" y2="124.46" width="0.1524" layer="91"/>
 <wire x1="76.2" y1="124.46" x2="76.2" y2="137.16" width="0.1524" layer="91"/>
 <wire x1="76.2" y1="137.16" x2="76.2" y2="142.24" width="0.1524" layer="91"/>
-<wire x1="83.82" y1="137.16" x2="76.2" y2="137.16" width="0.1524" layer="91"/>
+<wire x1="83.82" y1="137.16" x2="81.28" y2="137.16" width="0.1524" layer="91"/>
 <junction x="76.2" y="137.16"/>
-<wire x1="83.82" y1="116.84" x2="76.2" y2="116.84" width="0.1524" layer="91"/>
+<wire x1="81.28" y1="137.16" x2="76.2" y2="137.16" width="0.1524" layer="91"/>
+<wire x1="83.82" y1="116.84" x2="81.28" y2="116.84" width="0.1524" layer="91"/>
+<wire x1="81.28" y1="116.84" x2="76.2" y2="116.84" width="0.1524" layer="91"/>
 <wire x1="76.2" y1="116.84" x2="76.2" y2="119.38" width="0.1524" layer="91"/>
 <junction x="76.2" y="124.46"/>
 <wire x1="76.2" y1="119.38" x2="76.2" y2="121.92" width="0.1524" layer="91"/>
 <wire x1="76.2" y1="121.92" x2="76.2" y2="124.46" width="0.1524" layer="91"/>
-<wire x1="83.82" y1="114.3" x2="76.2" y2="114.3" width="0.1524" layer="91"/>
+<wire x1="83.82" y1="114.3" x2="81.28" y2="114.3" width="0.1524" layer="91"/>
+<wire x1="81.28" y1="114.3" x2="76.2" y2="114.3" width="0.1524" layer="91"/>
 <wire x1="76.2" y1="114.3" x2="76.2" y2="116.84" width="0.1524" layer="91"/>
-<wire x1="83.82" y1="119.38" x2="76.2" y2="119.38" width="0.1524" layer="91"/>
+<wire x1="83.82" y1="119.38" x2="81.28" y2="119.38" width="0.1524" layer="91"/>
 <pinref part="U$1" gate="G$1" pin="VCC1"/>
+<wire x1="81.28" y1="119.38" x2="76.2" y2="119.38" width="0.1524" layer="91"/>
 <wire x1="81.28" y1="121.92" x2="76.2" y2="121.92" width="0.1524" layer="91"/>
 <junction x="76.2" y="116.84"/>
@@
 <pinref part="C3" gate="G$1" pin="2"/>
 <wire x1="76.2" y1="121.92" x2="68.58" y2="121.92" width="0.1524" layer="91"/>
+<pinref part="U$1" gate="G$1" pin="/RESET"/>
+<junction x="81.28" y="137.16"/>
+<pinref part="U$1" gate="G$1" pin="VCC"/>
+<junction x="81.28" y="124.46"/>
+<junction x="81.28" y="121.92"/>
+<pinref part="U$1" gate="G$1" pin="UVCC"/>
+<junction x="81.28" y="119.38"/>
+<pinref part="U$1" gate="G$1" pin="AVCC"/>
+<junction x="81.28" y="116.84"/>
+<pinref part="U$1" gate="G$1" pin="AVCC1"/>
+<junction x="81.28" y="114.3"/>
 </segment>
 <segment>
@@
 <wire x1="81.28" y1="132.08" x2="63.5" y2="132.08" width="0.1524" layer="91"/>
 <label x="63.5" y="132.08" size="1.778" layer="95"/>
-</segment>
-<segment>
+<junction x="81.28" y="132.08"/>
+</segment>
+<segment>

Commit message: Finished micro and adjusted text of accel
MUST CHECK THAT TPLACE IS ON SILSCREEN OR SHIT!!!
Parts:
- renumbered C1 to C101, C2 to C102, C3 to C103, C4 to C104, JP1 to USB-UB, R1 to R101, R2 to R102, R3 to R103, R4 to R104, R5 to R105
