File: Hardware/power_RevA/Power_RevA.brd (EAGLE design)
At the start: 160 x 100 mm, 11 parts, among them Q401 TIP120

Commit message: Centered it to fit in 5cm x 5cm
And am going to CAM it.
Parts:
- moved C401 26.4 mm to (27.3, 41.2)
- moved LED2 26.4 mm to (25.1, 43.0)
- moved ACCEL 26.4 mm to (25.0, 35.7)
- moved C402 26.4 mm to (22.9, 41.3)
- moved LED1 26.4 mm to (10.5, 15.4)
- moved LED3 26.4 mm to (39.4, 15.0)
- moved MICRO 26.4 mm to (15.8, 20.8)
- moved PWR_IN 26.4 mm to (26.5, 13.4)
- moved Q401 26.4 mm to (18.8, 27.8)
- moved TOUCH 26.4 mm to (34.0, 20.2)
- moved TO_PAD 26.4 mm to (30.4, 29.2)
Other:
- board size 160 x 100 mm -> 51 x 50 mm

Commit message: More adjustments
Other:
- board size 51 x 50 mm -> 50 x 50 mm
Changed lines of the file:
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@@
 <wire x1="0" y1="0" x2="50" y2="0" width="0" layer="20"/>
 <wire x1="50" y1="0" x2="50" y2="50" width="0" layer="20"/>
-<wire x1="50" y1="50" x2="-1" y2="50" width="0" layer="20"/>
-<wire x1="-1" y1="50" x2="0" y2="0" width="0" layer="20"/>
+<wire x1="50" y1="50" x2="0" y2="50" width="0" layer="20"/>
+<wire x1="0" y1="50" x2="0" y2="0" width="0" layer="20"/>
 <circle x="25.1" y="25.26" radius="24.384" width="0.4064" layer="16"/>
 <text x="26.7002" y="10.0708" size="1.778" layer="21" rot="MR315">+</text>
