File: Hardware/power_RevA/Power_RevA.sch (EAGLE design)
At the start: 11 parts, among them Q1 TIP120

Commit message: Added labels, resized boundary
Everything is labeled now, but the boards needs to be placed in the 5cm
by 5cm boundary. The vias leave their holes behind though....
Parts:
- renumbered ACC to ACCEL, C1 to C401, C2 to C402, POWER to PWR_IN, Q1 to Q401, TOUCHSENSOR to TO_PAD
Changed lines of the file:
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@@
 <part name="MICRO" library="pinhead" deviceset="PINHD-1X6" device=""/>
 <part name="TOUCH" library="pinhead" deviceset="PINHD-1X4" device=""/>
-<part name="ACC" library="pinhead" deviceset="PINHD-1X3" device=""/>
-<part name="POWER" library="pinhead" deviceset="PINHD-1X2" device=""/>
-<part name="TOUCHSENSOR" library="pinhead" deviceset="PINHD-1X1" device=""/>
-<part name="Q1" library="transistor-power" deviceset="TIP120" device=""/>
+<part name="ACCEL" library="pinhead" deviceset="PINHD-1X3" device=""/>
+<part name="PWR_IN" library="pinhead" deviceset="PINHD-1X2" device=""/>
+<part name="TO_PAD" library="pinhead" deviceset="PINHD-1X1" device=""/>
+<part name="Q401" library="transistor-power" deviceset="TIP120" device=""/>
 <part name="LED1" library="led" deviceset="LED" device="P-LCC-4"/>
 <part name="LED2" library="led" deviceset="LED" device="P-LCC-4"/>
 <part name="LED3" library="led" deviceset="LED" device="P-LCC-4"/>
-<part name="C1" library="eagle-ltspice" deviceset="C" device="C0603" value="100n"/>
-<part name="C2" library="eagle-ltspice" deviceset="C" device="C0603" value="10u"/>
+<part name="C401" library="eagle-ltspice" deviceset="C" device="C0603" value="100n"/>
+<part name="C402" library="eagle-ltspice" deviceset="C" device="C0603" value="10u"/>
 </parts>
 <sheets>
@@
 <instance part="MICRO" gate="A" x="106.68" y="71.12"/>
 <instance part="TOUCH" gate="A" x="106.68" y="35.56"/>
-<instance part="ACC" gate="A" x="106.68" y="7.62"/>
-<instance part="POWER" gate="G$1" x="48.26" y="20.32"/>
-<instance part="TOUCHSENSOR" gate="G$1" x="86.36" y="33.02"/>
-<instance part="Q1" gate="1" x="55.88" y="58.42" rot="R180"/>
+<instance part="ACCEL" gate="A" x="106.68" y="7.62"/>
+<instance part="PWR_IN" gate="G$1" x="48.26" y="20.32"/>
+<instance part="TO_PAD" gate="G$1" x="86.36" y="33.02"/>
+<instance part="Q401" gate="1" x="55.88" y="58.42" rot="R180"/>
 <instance part="LED1" gate="G$1" x="20.32" y="63.5"/>
 <instance part="LED2" gate="G$1" x="10.16" y="63.5"/>
 <instance part="LED3" gate="G$1" x="-5.08" y="63.5"/>
-<instance part="C1" gate="G$1" x="38.1" y="53.34"/>
-<instance part="C2" gate="G$1" x="76.2" y="63.5" rot="R90"/>
+<instance part="C401" gate="G$1" x="38.1" y="53.34"/>
+<instance part="C402" gate="G$1" x="76.2" y="63.5" rot="R90"/>
 </instances>
 <busses>
@@
 <wire x1="91.44" y1="25.4" x2="78.74" y2="25.4" width="0.1524" layer="91"/>
 <wire x1="78.74" y1="25.4" x2="78.74" y2="33.02" width="0.1524" layer="91"/>
-<pinref part="TOUCHSENSOR" gate="G$1" pin="1"/>
+<pinref part="TO_PAD" gate="G$1" pin="1"/>
 <wire x1="78.74" y1="33.02" x2="83.82" y2="33.02" width="0.1524" layer="91"/>
 </segment>
@@
 <net name="N$2" class="0">
 <segment>
-<pinref part="POWER" gate="G$1" pin="1"/>
+<pinref part="PWR_IN" gate="G$1" pin="1"/>
 <wire x1="45.72" y1="22.86" x2="35.56" y2="22.86" width="0.1524" layer="91"/>
 <wire x1="35.56" y1="22.86" x2="35.56" y2="45.72" width="0.1524" layer="91"/>
@@
 <wire x1="63.5" y1="40.64" x2="63.5" y2="45.72" width="0.1524" layer="91"/>
 <junction x="63.5" y="45.72"/>
-<pinref part="ACC" gate="A" pin="1"/>
+<pinref part="ACCEL" gate="A" pin="1"/>
 <wire x1="104.14" y1="10.16" x2="88.9" y2="10.16" width="0.1524" layer="91"/>
 <wire x1="88.9" y1="10.16" x2="88.9" y2="40.64" width="0.1524" layer="91"/>
 <junction x="88.9" y="40.64"/>
-<pinref part="C1" gate="G$1" pin="2"/>
+<pinref part="C401" gate="G$1" pin="2"/>
 <wire x1="38.1" y1="48.26" x2="38.1" y2="45.72" width="0.1524" layer="91"/>
 <junction x="38.1" y="45.72"/>
-<pinref part="Q1" gate="1" pin="E"/>
+<pinref part="Q401" gate="1" pin="E"/>
 <wire x1="53.34" y1="63.5" x2="48.26" y2="63.5" width="0.1524" layer="91"/>
 <wire x1="48.26" y1="63.5" x2="48.26" y2="45.72" width="0.1524" layer="91"/>
@@
 <wire x1="104.14" y1="38.1" x2="93.98" y2="38.1" width="0.1524" layer="91"/>
 <wire x1="93.98" y1="38.1" x2="93.98" y2="58.42" width="0.1524" layer="91"/>
-<pinref part="ACC" gate="A" pin="2"/>
+<pinref part="ACCEL" gate="A" pin="2"/>
 <wire x1="93.98" y1="58.42" x2="93.98" y2="63.5" width="0.1524" layer="91"/>
 <wire x1="104.14" y1="7.62" x2="93.98" y2="7.62" width="0.1524" layer="91"/>
 <wire x1="93.98" y1="7.62" x2="93.98" y2="38.1" width="0.1524" layer="91"/>
 <junction x="93.98" y="38.1"/>
-<pinref part="C2" gate="G$1" pin="2"/>
+<pinref part="C402" gate="G$1" pin="2"/>
 <wire x1="81.28" y1="63.5" x2="93.98" y2="63.5" width="0.1524" layer="91"/>
 <junction x="93.98" y="63.5"/>
@@
 <wire x1="66.04" y1="58.42" x2="93.98" y2="58.42" width="0.1524" layer="91"/>
 <junction x="93.98" y="58.42"/>
-<pinref part="Q1" gate="1" pin="C"/>
+<pinref part="Q401" gate="1" pin="C"/>
 <wire x1="53.34" y1="53.34" x2="53.34" y2="48.26" width="0.1524" layer="91"/>
 <wire x1="53.34" y1="48.26" x2="60.96" y2="48.26" width="0.1524" layer="91"/>
@@
 <wire x1="99.06" y1="35.56" x2="99.06" y2="53.34" width="0.1524" layer="91"/>
 <junction x="99.06" y="35.56"/>
-<pinref part="ACC" gate="A" pin="3"/>
+<pinref part="ACCEL" gate="A" pin="3"/>
 <wire x1="99.06" y1="53.34" x2="99.06" y2="73.66" width="0.1524" layer="91"/>
 <wire x1="104.14" y1="5.08" x2="99.06" y2="5.08" width="0.1524" layer="91"/>
 <wire x1="99.06" y1="5.08" x2="99.06" y2="35.56" width="0.1524" layer="91"/>
-<pinref part="C2" gate="G$1" pin="1"/>
+<pinref part="C402" gate="G$1" pin="1"/>
 <wire x1="73.66" y1="63.5" x2="68.58" y2="63.5" width="0.1524" layer="91"/>
 <wire x1="68.58" y1="63.5" x2="68.58" y2="73.66" width="0.1524" layer="91"/>
@@
 <wire x1="38.1" y1="63.5" x2="30.48" y2="63.5" width="0.1524" layer="91"/>
 <wire x1="30.48" y1="63.5" x2="30.48" y2="35.56" width="0.1524" layer="91"/>
-<pinref part="POWER" gate="G$1" pin="2"/>
+<pinref part="PWR_IN" gate="G$1" pin="2"/>
 <wire x1="30.48" y1="35.56" x2="30.48" y2="20.32" width="0.1524" layer="91"/>
 <wire x1="30.48" y1="20.32" x2="45.72" y2="20.32" width="0.1524" layer="91"/>
@@
 <wire x1="-5.08" y1="35.56" x2="10.16" y2="35.56" width="0.1524" layer="91"/>
 <junction x="10.16" y="35.56"/>
-<pinref part="C1" gate="G$1" pin="1"/>
+<pinref part="C401" gate="G$1" pin="1"/>
 <wire x1="38.1" y1="55.88" x2="38.1" y2="63.5" width="0.1524" layer="91"/>
 <wire x1="71.12" y1="81.28" x2="30.48" y2="81.28" width="0.1524" layer="91"/>
 <wire x1="30.48" y1="81.28" x2="30.48" y2="63.5" width="0.1524" layer="91"/>
 <junction x="30.48" y="63.5"/>
-<pinref part="Q1" gate="1" pin="B"/>
+<pinref part="Q401" gate="1" pin="B"/>
 <wire x1="99.06" y1="53.34" x2="58.42" y2="53.34" width="0.1524" layer="91"/>
 <wire x1="58.42" y1="53.34" x2="58.42" y2="58.42" width="0.1524" layer="91"/>

Commit message: Power and Touch Board LED Orientation Fixed
The touch board is sill routed incorrectly (schematic is wrong too) but
orientation is silk-screened on board. Power board is routed absolutely
correctly.
Connections:
- removed net N$7: LED1.A, MICRO.6
- new net N$3: LED1.C, MICRO.6
- net N$2: now also LED1.A, LED2.A, LED3.A
- net N$5: now also LED2.C, MICRO.5; no longer LED3.A, MICRO.4
- net N$6: now also LED3.C, MICRO.4; no longer LED2.A, MICRO.5
- net N$8: no longer LED1.C, LED2.C, LED3.C
Other:
- moved on the sheet: LED1, LED2, LED3
Changed lines of the file:
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@@
 <instance part="TO_PAD" gate="G$1" x="86.36" y="33.02"/>
 <instance part="Q401" gate="1" x="55.88" y="58.42" rot="R180"/>
-<instance part="LED1" gate="G$1" x="20.32" y="63.5"/>
-<instance part="LED2" gate="G$1" x="10.16" y="63.5"/>
-<instance part="LED3" gate="G$1" x="-5.08" y="63.5"/>
+<instance part="LED1" gate="G$1" x="20.32" y="53.34" rot="R180"/>
+<instance part="LED2" gate="G$1" x="10.16" y="53.34" rot="R180"/>
+<instance part="LED3" gate="G$1" x="0" y="53.34" rot="R180"/>
 <instance part="C401" gate="G$1" x="38.1" y="53.34"/>
 <instance part="C402" gate="G$1" x="76.2" y="63.5" rot="R90"/>
@@
 <pinref part="PWR_IN" gate="G$1" pin="1"/>
 <wire x1="45.72" y1="22.86" x2="35.56" y2="22.86" width="0.1524" layer="91"/>
-<wire x1="35.56" y1="22.86" x2="35.56" y2="45.72" width="0.1524" layer="91"/>
+<wire x1="35.56" y1="22.86" x2="35.56" y2="35.56" width="0.1524" layer="91"/>
+<wire x1="35.56" y1="35.56" x2="35.56" y2="45.72" width="0.1524" layer="91"/>
 <wire x1="35.56" y1="45.72" x2="38.1" y2="45.72" width="0.1524" layer="91"/>
 <wire x1="38.1" y1="45.72" x2="48.26" y2="45.72" width="0.1524" layer="91"/>
@@
 <wire x1="48.26" y1="63.5" x2="48.26" y2="45.72" width="0.1524" layer="91"/>
 <junction x="48.26" y="45.72"/>
+<pinref part="LED1" gate="G$1" pin="A"/>
+<wire x1="20.32" y1="50.8" x2="20.32" y2="38.1" width="0.1524" layer="91"/>
+<wire x1="20.32" y1="38.1" x2="20.32" y2="35.56" width="0.1524" layer="91"/>
+<wire x1="20.32" y1="35.56" x2="35.56" y2="35.56" width="0.1524" layer="91"/>
+<junction x="35.56" y="35.56"/>
+<pinref part="LED2" gate="G$1" pin="A"/>
+<wire x1="10.16" y1="50.8" x2="10.16" y2="40.64" width="0.1524" layer="91"/>
+<wire x1="10.16" y1="40.64" x2="10.16" y2="38.1" width="0.1524" layer="91"/>
+<wire x1="10.16" y1="38.1" x2="20.32" y2="38.1" width="0.1524" layer="91"/>
+<junction x="20.32" y="38.1"/>
+<pinref part="LED3" gate="G$1" pin="A"/>
+<wire x1="0" y1="50.8" x2="0" y2="40.64" width="0.1524" layer="91"/>
+<wire x1="0" y1="40.64" x2="10.16" y2="40.64" width="0.1524" layer="91"/>
+<junction x="10.16" y="40.64"/>
 </segment>
 </net>
@@
 </segment>
 </net>
-<net name="N$5" class="0">
-<segment>
-<pinref part="MICRO" gate="A" pin="4"/>
-<pinref part="LED3" gate="G$1" pin="A"/>
-<wire x1="104.14" y1="71.12" x2="-5.08" y2="71.12" width="0.1524" layer="91"/>
-<wire x1="-5.08" y1="71.12" x2="-5.08" y2="66.04" width="0.1524" layer="91"/>
-</segment>
-</net>
-<net name="N$6" class="0">
-<segment>
-<pinref part="MICRO" gate="A" pin="5"/>
-<pinref part="LED2" gate="G$1" pin="A"/>
-<wire x1="104.14" y1="68.58" x2="10.16" y2="68.58" width="0.1524" layer="91"/>
-<wire x1="10.16" y1="68.58" x2="10.16" y2="66.04" width="0.1524" layer="91"/>
-</segment>
-</net>
-<net name="N$7" class="0">
-<segment>
-<pinref part="MICRO" gate="A" pin="6"/>
-<pinref part="LED1" gate="G$1" pin="A"/>
-<wire x1="104.14" y1="66.04" x2="20.32" y2="66.04" width="0.1524" layer="91"/>
-</segment>
-</net>
 <net name="N$8" class="0">
 <segment>
@@
 <junction x="71.12" y="73.66"/>
 <wire x1="38.1" y1="63.5" x2="30.48" y2="63.5" width="0.1524" layer="91"/>
-<wire x1="30.48" y1="63.5" x2="30.48" y2="35.56" width="0.1524" layer="91"/>
+<wire x1="30.48" y1="63.5" x2="30.48" y2="20.32" width="0.1524" layer="91"/>
 <pinref part="PWR_IN" gate="G$1" pin="2"/>
-<wire x1="30.48" y1="35.56" x2="30.48" y2="20.32" width="0.1524" layer="91"/>
 <wire x1="30.48" y1="20.32" x2="45.72" y2="20.32" width="0.1524" layer="91"/>
-<pinref part="LED1" gate="G$1" pin="C"/>
-<wire x1="20.32" y1="58.42" x2="20.32" y2="35.56" width="0.1524" layer="91"/>
-<wire x1="20.32" y1="35.56" x2="30.48" y2="35.56" width="0.1524" layer="91"/>
-<junction x="30.48" y="35.56"/>
-<pinref part="LED2" gate="G$1" pin="C"/>
-<wire x1="10.16" y1="58.42" x2="10.16" y2="35.56" width="0.1524" layer="91"/>
-<wire x1="10.16" y1="35.56" x2="20.32" y2="35.56" width="0.1524" layer="91"/>
-<junction x="20.32" y="35.56"/>
-<pinref part="LED3" gate="G$1" pin="C"/>
-<wire x1="-5.08" y1="58.42" x2="-5.08" y2="35.56" width="0.1524" layer="91"/>
-<wire x1="-5.08" y1="35.56" x2="10.16" y2="35.56" width="0.1524" layer="91"/>
-<junction x="10.16" y="35.56"/>
 <pinref part="C401" gate="G$1" pin="1"/>
 <wire x1="38.1" y1="55.88" x2="38.1" y2="63.5" width="0.1524" layer="91"/>
@@
 </segment>
 </net>
+<net name="N$3" class="0">
+<segment>
+<pinref part="LED1" gate="G$1" pin="C"/>
+<pinref part="MICRO" gate="A" pin="6"/>
+<wire x1="20.32" y1="58.42" x2="20.32" y2="66.04" width="0.1524" layer="91"/>
+<wire x1="20.32" y1="66.04" x2="104.14" y2="66.04" width="0.1524" layer="91"/>
+</segment>
+</net>
+<net name="N$5" class="0">
+<segment>
+<pinref part="LED2" gate="G$1" pin="C"/>
+<pinref part="MICRO" gate="A" pin="5"/>
+<wire x1="10.16" y1="58.42" x2="10.16" y2="68.58" width="0.1524" layer="91"/>
+<wire x1="10.16" y1="68.58" x2="104.14" y2="68.58" width="0.1524" layer="91"/>
+</segment>
+</net>
+<net name="N$6" class="0">
+<segment>
+<pinref part="LED3" gate="G$1" pin="C"/>
+<pinref part="MICRO" gate="A" pin="4"/>
+<wire x1="0" y1="58.42" x2="0" y2="71.12" width="0.1524" layer="91"/>
+<wire x1="0" y1="71.12" x2="104.14" y2="71.12" width="0.1524" layer="91"/>
+</segment>
+</net>

Commit message: Added Javen's logo to everything
Still need to add plus/minus on leds before order.
Connections:
- removed net N$3: LED1.C, MICRO.6
- new net N$7: LED1.A, MICRO.6
- net N$2: no longer LED1.A, LED2.A, LED3.A
- net N$5: now also LED3.A, MICRO.4; no longer LED2.C, MICRO.5
- net N$6: now also LED2.A, MICRO.5; no longer LED3.C, MICRO.4
- net N$8: now also LED1.C, LED2.C, LED3.C
Other:
- moved on the sheet: LED1, LED2, LED3
Changed lines of the file:
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@@
 <instance part="TO_PAD" gate="G$1" x="86.36" y="33.02"/>
 <instance part="Q401" gate="1" x="55.88" y="58.42" rot="R180"/>
-<instance part="LED1" gate="G$1" x="20.32" y="53.34" rot="R180"/>
-<instance part="LED2" gate="G$1" x="10.16" y="53.34" rot="R180"/>
-<instance part="LED3" gate="G$1" x="0" y="53.34" rot="R180"/>
+<instance part="LED1" gate="G$1" x="20.32" y="63.5"/>
+<instance part="LED2" gate="G$1" x="10.16" y="63.5"/>
+<instance part="LED3" gate="G$1" x="-5.08" y="63.5"/>
 <instance part="C401" gate="G$1" x="38.1" y="53.34"/>
 <instance part="C402" gate="G$1" x="76.2" y="63.5" rot="R90"/>
@@
 <pinref part="PWR_IN" gate="G$1" pin="1"/>
 <wire x1="45.72" y1="22.86" x2="35.56" y2="22.86" width="0.1524" layer="91"/>
-<wire x1="35.56" y1="22.86" x2="35.56" y2="35.56" width="0.1524" layer="91"/>
-<wire x1="35.56" y1="35.56" x2="35.56" y2="45.72" width="0.1524" layer="91"/>
+<wire x1="35.56" y1="22.86" x2="35.56" y2="45.72" width="0.1524" layer="91"/>
 <wire x1="35.56" y1="45.72" x2="38.1" y2="45.72" width="0.1524" layer="91"/>
 <wire x1="38.1" y1="45.72" x2="48.26" y2="45.72" width="0.1524" layer="91"/>
@@
 <wire x1="48.26" y1="63.5" x2="48.26" y2="45.72" width="0.1524" layer="91"/>
 <junction x="48.26" y="45.72"/>
-<pinref part="LED1" gate="G$1" pin="A"/>
-<wire x1="20.32" y1="50.8" x2="20.32" y2="38.1" width="0.1524" layer="91"/>
-<wire x1="20.32" y1="38.1" x2="20.32" y2="35.56" width="0.1524" layer="91"/>
-<wire x1="20.32" y1="35.56" x2="35.56" y2="35.56" width="0.1524" layer="91"/>
-<junction x="35.56" y="35.56"/>
-<pinref part="LED2" gate="G$1" pin="A"/>
-<wire x1="10.16" y1="50.8" x2="10.16" y2="40.64" width="0.1524" layer="91"/>
-<wire x1="10.16" y1="40.64" x2="10.16" y2="38.1" width="0.1524" layer="91"/>
-<wire x1="10.16" y1="38.1" x2="20.32" y2="38.1" width="0.1524" layer="91"/>
-<junction x="20.32" y="38.1"/>
-<pinref part="LED3" gate="G$1" pin="A"/>
-<wire x1="0" y1="50.8" x2="0" y2="40.64" width="0.1524" layer="91"/>
-<wire x1="0" y1="40.64" x2="10.16" y2="40.64" width="0.1524" layer="91"/>
-<junction x="10.16" y="40.64"/>
 </segment>
 </net>
@@
 </segment>
 </net>
+<net name="N$5" class="0">
+<segment>
+<pinref part="MICRO" gate="A" pin="4"/>
+<pinref part="LED3" gate="G$1" pin="A"/>
+<wire x1="104.14" y1="71.12" x2="-5.08" y2="71.12" width="0.1524" layer="91"/>
+<wire x1="-5.08" y1="71.12" x2="-5.08" y2="66.04" width="0.1524" layer="91"/>
+</segment>
+</net>
+<net name="N$6" class="0">
+<segment>
+<pinref part="MICRO" gate="A" pin="5"/>
+<pinref part="LED2" gate="G$1" pin="A"/>
+<wire x1="104.14" y1="68.58" x2="10.16" y2="68.58" width="0.1524" layer="91"/>
+<wire x1="10.16" y1="68.58" x2="10.16" y2="66.04" width="0.1524" layer="91"/>
+</segment>
+</net>
+<net name="N$7" class="0">
+<segment>
+<pinref part="MICRO" gate="A" pin="6"/>
+<pinref part="LED1" gate="G$1" pin="A"/>
+<wire x1="104.14" y1="66.04" x2="20.32" y2="66.04" width="0.1524" layer="91"/>
+</segment>
+</net>
 <net name="N$8" class="0">
 <segment>
@@
 <junction x="71.12" y="73.66"/>
 <wire x1="38.1" y1="63.5" x2="30.48" y2="63.5" width="0.1524" layer="91"/>
-<wire x1="30.48" y1="63.5" x2="30.48" y2="20.32" width="0.1524" layer="91"/>
+<wire x1="30.48" y1="63.5" x2="30.48" y2="35.56" width="0.1524" layer="91"/>
 <pinref part="PWR_IN" gate="G$1" pin="2"/>
+<wire x1="30.48" y1="35.56" x2="30.48" y2="20.32" width="0.1524" layer="91"/>
 <wire x1="30.48" y1="20.32" x2="45.72" y2="20.32" width="0.1524" layer="91"/>
+<pinref part="LED1" gate="G$1" pin="C"/>
+<wire x1="20.32" y1="58.42" x2="20.32" y2="35.56" width="0.1524" layer="91"/>
+<wire x1="20.32" y1="35.56" x2="30.48" y2="35.56" width="0.1524" layer="91"/>
+<junction x="30.48" y="35.56"/>
+<pinref part="LED2" gate="G$1" pin="C"/>
+<wire x1="10.16" y1="58.42" x2="10.16" y2="35.56" width="0.1524" layer="91"/>
+<wire x1="10.16" y1="35.56" x2="20.32" y2="35.56" width="0.1524" layer="91"/>
+<junction x="20.32" y="35.56"/>
+<pinref part="LED3" gate="G$1" pin="C"/>
+<wire x1="-5.08" y1="58.42" x2="-5.08" y2="35.56" width="0.1524" layer="91"/>
+<wire x1="-5.08" y1="35.56" x2="10.16" y2="35.56" width="0.1524" layer="91"/>
+<junction x="10.16" y="35.56"/>
 <pinref part="C401" gate="G$1" pin="1"/>
 <wire x1="38.1" y1="55.88" x2="38.1" y2="63.5" width="0.1524" layer="91"/>
@@
 </segment>
 </net>
-<net name="N$3" class="0">
-<segment>
-<pinref part="LED1" gate="G$1" pin="C"/>
-<pinref part="MICRO" gate="A" pin="6"/>
-<wire x1="20.32" y1="58.42" x2="20.32" y2="66.04" width="0.1524" layer="91"/>
-<wire x1="20.32" y1="66.04" x2="104.14" y2="66.04" width="0.1524" layer="91"/>
-</segment>
-</net>
-<net name="N$5" class="0">
-<segment>
-<pinref part="LED2" gate="G$1" pin="C"/>
-<pinref part="MICRO" gate="A" pin="5"/>
-<wire x1="10.16" y1="58.42" x2="10.16" y2="68.58" width="0.1524" layer="91"/>
-<wire x1="10.16" y1="68.58" x2="104.14" y2="68.58" width="0.1524" layer="91"/>
-</segment>
-</net>
-<net name="N$6" class="0">
-<segment>
-<pinref part="LED3" gate="G$1" pin="C"/>
-<pinref part="MICRO" gate="A" pin="4"/>
-<wire x1="0" y1="58.42" x2="0" y2="71.12" width="0.1524" layer="91"/>
-<wire x1="0" y1="71.12" x2="104.14" y2="71.12" width="0.1524" layer="91"/>
-</segment>
-</net>
