File: Hardware/accel_RevA/accel_RevA.brd (EAGLE design)
At the start: 50.3 x 50 mm, 12 parts, among them U1 MMA8452Q

Commit message: Added Javen's logo to everything
Still need to add plus/minus on leds before order.
Other:
- board text added: "v0.1"
- board text removed: "TES"

Commit message: Update of hw files
Added logo to brds, added +/- to LEDs and generated and updated gerber
files.
Other:
- board size 50.3 x 50 mm -> 49.9 x 50 mm
- board text added: "+"
- board text added: "-"
